Commit message: openarm01_arm: move to a non-singular ready pose on startup; raise elbow floor
The arm powers off wherever it hung, often with the elbow near-straight, which is
the arm-angle IK's one true singularity (shoulder, elbow, wrist colinear, so the
arm angle is undefined). Starting a Cartesian move from there is ill-posed.

Add a Startup state, the machine's first: it eases from the measured power-on
configuration to a fixed non-singular ready pose (elbow bent a hair off the
singularity) with a gentle joint trajectory, then transitions to Hold. The
single-flight flag is born held and released only when Startup reaches the ready
pose, so a goal arriving during startup is rejected as busy rather than queued
behind a motion the caller never requested.

Raise the J4 (elbow) lower limit in the description URDF from the vendored 0.0 to
0.05 rad so neither the IK nor joint-target validation can command full extension.
Pick up the merged srs_model arm-angle fix via Cargo.lock.

File: description/openarm_v10.urdf (robot description, URDF)
Before this commit: robot openarm, 24 links, 23 joints
Joints:
- joint openarm_left_joint4: limit lower=0.0 upper=2.443461 effort=27 velocity=5.445426 -> lower=0.05 upper=2.443461 effort=27 velocity=5.445426
- joint openarm_right_joint4: limit lower=0.0 upper=2.443461 effort=27 velocity=5.445426 -> lower=0.05 upper=2.443461 effort=27 velocity=5.445426
